Commit message: chaned fiel paths in .urdf

File: src/description/urdf/arduinobot.urdf (robot description, URDF)
Before this commit: robot arduinobot, 8 links, 7 joints
Links:
- link base_link: geometry collision mesh filename=../meshes/basement.STL scale=0.01 0.01 0.01; visual mesh filename=../meshes/basement.STL scale=0.01 0.01 0.01
- link base_plate: geometry collision mesh filename=../meshes/base_plate.STL scale=0.01 0.01 0.01; visual mesh filename=../meshes/base_plate.STL scale=0.01 0.01 0.01
- link claw_support: geometry collision mesh filename=../meshes/claw_support.STL scale=0.01 0.01 0.01; visual mesh filename=../meshes/claw_support.STL scale=0.01 0.01 0.01
- link forward_drive_arm: geometry collision mesh filename=../meshes/forward_drive_arm.STL scale=0.01 0.01 0.01; visual mesh filename=../meshes/forward_drive_arm.STL scale=0.01 0.01 0.01
- link gripper_left: geometry collision mesh filename=../meshes/left_finger.STL scale=0.01 0.01 0.01; visual mesh filename=../meshes/left_finger.STL scale=0.01 0.01 0.01
- link gripper_right: geometry collision mesh filename=../meshes/right_finger.STL scale=0.01 0.01 0.01; visual mesh filename=../meshes/right_finger.STL scale=0.01 0.01 0.01
- link horizontal_arm: geometry collision mesh filename=../meshes/horizontal_arm.STL scale=0.01 0.01 0.01; visual mesh filename=../meshes/horizontal_arm.STL scale=0.01 0.01 0.01

Commit message: modified .urdf to support absolute paths

File: src/description/urdf/arduinobot.urdf (robot description, URDF)
Before this commit: robot arduinobot, 8 links, 7 joints
Links:
- link base_link: geometry collision mesh filename=/home/shourya/mujoco_ws/src/description/meshes/basement.STL scale=0.01 0.01 0.01; visual mesh filename=/home/shourya/mujoco_ws/src/description/meshes/basement.STL scale=0.01 0.01 0.01
- link base_plate: geometry collision mesh filename=/home/shourya/mujoco_ws/src/description/meshes/base_plate.S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 scale=0.01 0.01 0.01; visual mesh filename=/home/shourya/mujoco_ws/src/description/meshes/base_plate.S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 scale=0.01 0.01 0.01
- link claw_support: geometry collision mesh filename=/home/shourya/mujoco_ws/src/description/meshes/claw_support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 scale=0.01 0.01 0.01; visual mesh filename=/home/shourya/mujoco_ws/src/description/meshes/claw_support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 scale=0.01 0.01 0.01
- link forward_drive_arm: geometry collision mesh filename=/home/shourya/mujoco_ws/src/description/meshes/forward_driv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 scale=0.01 0.01 0.01; visual mesh filename=/home/shourya/mujoco_ws/src/description/meshes/forward_driv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 scale=0.01 0.01 0.01
- link gripper_left: geometry collision mesh filename=/home/shourya/mujoco_ws/src/description/meshes/left_finger.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 scale=0.01 0.01 0.01; visual mesh filename=/home/shourya/mujoco_ws/src/description/meshes/left_finger.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 scale=0.01 0.01 0.01
- link gripper_right: geometry collision mesh filename=/home/shourya/mujoco_ws/src/description/meshes/right_finger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 scale=0.01 0.01 0.01; visual mesh filename=/home/shourya/mujoco_ws/src/description/meshes/right_finger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 scale=0.01 0.01 0.01
- link horizontal_arm: geometry collision mesh filename=/home/shourya/mujoco_ws/src/description/meshes/horizontal_a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 scale=0.01 0.01 0.01; visual mesh filename=/home/shourya/mujoco_ws/src/description/meshes/horizontal_a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 scale=0.01 0.01 0.01
