Commit message: modify code to use absolute paths

File: src/description/urdf/model.urdf (robot description, URDF)
Before this commit: robot inverted_pendulum, 4 links, 3 joints
Links:
- link arm: geometry visual mesh filename=/home/shourya/mujoco_ws/src/description/meshes/arm.stl scale=0.001 0.001 0.001
- link base: geometry visual mesh filename=/home/shourya/mujoco_ws/src/description/meshes/base.stl scale=0.001 0.001 0.001
- link lid: geometry visual mesh filename=/home/shourya/mujoco_ws/src/description/meshes/lid.stl scale=0.001 0.001 0.001
- link pendulum: geometry visual mesh filename=/home/shourya/mujoco_ws/src/description/meshes/pendulum.stl scale=0.001 0.001 0.001
